File: PCBs/Version2/RatDBS.brd (EAGLE design)
At the start: 25.4 x 15.9 mm, 14 parts

Commit message: Changed some colors and labels, changed code directory structure, and added docs for RF430
Parts:
- C1_SUPPLY: value (none) -> 10uF
Changed lines of the file:
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@@
 <element name="MSP430" library="BiphasicBoard" package="20_PIN" value="" x="19.6215" y="6.2865" smashed="yes" rot="MR270"/>
 <element name="TS3A4751_0" library="BiphasicBoard" package="14_PIN" value="" x="5.3975" y="3.2385" smashed="yes" rot="MR180"/>
-<element name="C1_SUPPLY" library="resistor" package="C0603" value="" x="19.431" y="10.8585" smashed="yes" rot="MR180">
-<attribute name="VALUE" x="18.542" y="12.8905" size="1.27" layer="28" rot="MR180"/>
+<element name="C1_SUPPLY" library="resistor" package="C0603" value="10uF" x="19.431" y="10.8585" smashed="yes" rot="MR180">
+<attribute name="VALUE" x="14.605" y="11.4935" size="0.8128" layer="28" font="vector" ratio="15" rot="MR180"/>
 </element>
 <element name="LED6" library="SparkFun-LED" package="LED-1206" value="GREEN" x="21.3995" y="2.032" smashed="yes" rot="R180">
