File: PCBs/Current/RatDBS-Compact2032Battery.sch (EAGLE design)
At the start: 20 parts

Commit message: Added an error state until NFC is read correctly.
Parts:
- removed ANT: FTSH-102, Samtec50Mil:FTSH-102
- added L1: (no value), rcl:L-EUWE-TPC
- C1: value 1µ -> 1u
- C2: value 0.1µ -> 0.1u
- CBAT: value 10µ -> 10u; device rcl:C-EUC1206 -> rcl:C-EUC0603
- C_VC: value 0.47µ -> 0.47u
Connections:
- net GND: now also CBAT.2; no longer CBAT.1
- net N$12: now also L1.2; no longer ANT.1
- net N$2: now also L1.1; no longer ANT.2
- net VDD: now also CBAT.1; no longer CBAT.2
Other:
- moved on the sheet: CBAT
Changed lines of the file:
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@@
 <part name="MSP430" library="RatDBS" deviceset="MSP430" device="" value="MSP"/>
 <part name="TS3A4751_0" library="BiphasicBoard" deviceset="TS3A4751" device="" value="SW"/>
-<part name="CBAT" library="rcl" deviceset="C-EU" device="C1206" value="10µ"/>
 <part name="LED6" library="SparkFun-LED" deviceset="LED" device="1206" value="GREEN"/>
 <part name="R_LOAD_EX" library="BiphasicBoard" deviceset="R-US_" device="R0603" value="10k"/>
@@
 <part name="GND9" library="supply1" deviceset="GND" device=""/>
 <part name="GND10" library="supply1" deviceset="GND" device=""/>
-<part name="C_VC" library="rcl" deviceset="C-EU" device="C0603" value="0.47µ"/>
-<part name="C2" library="rcl" deviceset="C-EU" device="C0603" value="0.1µ"/>
-<part name="ANT" library="Samtec50Mil" deviceset="FTSH-102" device=""/>
+<part name="C_VC" library="rcl" deviceset="C-EU" device="C0603" value="0.47u"/>
+<part name="C2" library="rcl" deviceset="C-EU" device="C0603" value="0.1u"/>
 <part name="CANT" library="rcl" deviceset="C-EU" device="C0603"/>
 <part name="BAT1" library="Battery" deviceset="BATTERY" device="FOB" value="20mm coincell"/>
 <part name="VDD11" library="supply1" deviceset="VDD" device=""/>
 <part name="GND11" library="supply1" deviceset="GND" device=""/>
-<part name="C1" library="rcl" deviceset="C-EU" device="C0603" value="1µ"/>
+<part name="C1" library="rcl" deviceset="C-EU" device="C0603" value="1u"/>
+<part name="L1" library="rcl" deviceset="L-EU" device="WE-TPC"/>
+<part name="CBAT" library="rcl" deviceset="C-EU" device="C0603" value="10u"/>
 </parts>
 <sheets>
@@
 <instance part="MSP430" gate="G$1" x="-20.32" y="73.66"/>
 <instance part="TS3A4751_0" gate="G$1" x="-25.4" y="27.94"/>
-<instance part="CBAT" gate="G$1" x="10.16" y="101.6" rot="R180"/>
 <instance part="LED6" gate="G$1" x="22.86" y="45.72"/>
 <instance part="R_LOAD_EX" gate="G$1" x="-63.5" y="7.62"/>
@@
 <instance part="C_VC" gate="G$1" x="-129.54" y="104.14" rot="R90"/>
 <instance part="C2" gate="G$1" x="-152.4" y="119.38" rot="R90"/>
-<instance part="ANT" gate="G$1" x="-195.58" y="101.6"/>
 <instance part="CANT" gate="G$1" x="-177.8" y="99.06" rot="R180"/>
 <instance part="BAT1" gate="G$1" x="-180.34" y="38.1" rot="R270"/>
@@
 <instance part="GND11" gate="1" x="-180.34" y="30.48"/>
 <instance part="C1" gate="G$1" x="-152.4" y="132.08" rot="R90"/>
+<instance part="L1" gate="G$1" x="-193.04" y="99.06"/>
+<instance part="CBAT" gate="G$1" x="10.16" y="104.14"/>
 </instances>
 <busses>
@@
 </segment>
 <segment>
-<pinref part="CBAT" gate="G$1" pin="2"/>
 <wire x1="10.16" y1="106.68" x2="10.16" y2="119.38" width="0.1524" layer="91"/>
 <pinref part="VDD1" gate="G$1" pin="VDD"/>
+<pinref part="CBAT" gate="G$1" pin="1"/>
 </segment>
 <segment>
@@
 <pinref part="GND7" gate="1" pin="GND"/>
 <wire x1="15.24" y1="83.82" x2="10.16" y2="81.28" width="0.1524" layer="91"/>
-<pinref part="CBAT" gate="G$1" pin="1"/>
 <wire x1="10.16" y1="81.28" x2="5.08" y2="81.28" width="0.1524" layer="91"/>
 <wire x1="10.16" y1="99.06" x2="10.16" y2="81.28" width="0.1524" layer="91"/>
 <junction x="10.16" y="81.28"/>
+<pinref part="CBAT" gate="G$1" pin="2"/>
 </segment>
 <segment>
@@
 <net name="N$2" class="0">
 <segment>
-<pinref part="ANT" gate="G$1" pin="2"/>
-<wire x1="-190.5" y1="101.6" x2="-185.42" y2="101.6" width="0.1524" layer="91"/>
-<wire x1="-185.42" y1="101.6" x2="-185.42" y2="104.14" width="0.1524" layer="91"/>
 <pinref part="CANT" gate="G$1" pin="2"/>
 <wire x1="-177.8" y1="104.14" x2="-185.42" y2="104.14" width="0.1524" layer="91"/>
@@
 <wire x1="-167.64" y1="104.14" x2="-177.8" y2="104.14" width="0.1524" layer="91"/>
 <junction x="-177.8" y="104.14"/>
+<pinref part="L1" gate="G$1" pin="1"/>
+<wire x1="-193.04" y1="104.14" x2="-193.04" y2="106.68" width="0.1524" layer="91"/>
+<wire x1="-193.04" y1="106.68" x2="-185.42" y2="106.68" width="0.1524" layer="91"/>
+<wire x1="-185.42" y1="106.68" x2="-185.42" y2="104.14" width="0.1524" layer="91"/>
 </segment>
 </net>
 <net name="N$12" class="0">
 <segment>
-<pinref part="ANT" gate="G$1" pin="1"/>
-<wire x1="-190.5" y1="99.06" x2="-185.42" y2="99.06" width="0.1524" layer="91"/>
-<wire x1="-185.42" y1="99.06" x2="-185.42" y2="96.52" width="0.1524" layer="91"/>
 <pinref part="CANT" gate="G$1" pin="1"/>
 <wire x1="-185.42" y1="96.52" x2="-177.8" y2="96.52" width="0.1524" layer="91"/>
@@
 <wire x1="-172.72" y1="96.52" x2="-177.8" y2="96.52" width="0.1524" layer="91"/>
 <junction x="-177.8" y="96.52"/>
-</segment>
-</net>
+<pinref part="L1" gate="G$1" pin="2"/>
+<wire x1="-193.04" y1="93.98" x2="-193.04" y2="91.44" width="0.1524" layer="91"/>
+<wire x1="-193.04" y1="91.44" x2="-185.42" y2="91.44" width="0.1524" layer="91"/>
+<wire x1="-185.42" y1="91.44" x2="-185.42" y2="96.52" width="0.1524" layer="91"/>
+</segment>
+</net>
