File: PCBs/Current/RatDBS-Plastic2032Battery-WithRegulator.brd (EAGLE design)
At the start: 28.3 x 22.9 mm, 23 parts, among them U1 LP2981-3V, U2 LP2981-5V

Commit message: Updated PCB manufacturing
Connections:
- removed net VDD2: C1.1, C2.1, U$1.1
- net VDD: now also C1.1, C2.1, U$1.1
Routing:
- net VDD: track 43.1 -> 60.9 mm, vias 3 -> 4
- net VDD2: track 5.28 -> 0.00 mm
- net GND: vias 8 -> 9
Other:
- board text added: "NFC-RDBS v2.1 Kemere Lab (C)2017"
- board text removed: "NFC-RDBS v2.0 Kemere Lab (C)2016"
Changed lines of the file:
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@@
 <?xml version="1.0" encoding="utf-8"?>
 <!DOCTYPE eagle SYSTEM "eagle.dtd">
-<eagle version="7.3.0">
+<eagle version="7.7.0">
 <drawing>
 <settings>
@@
 <wire x1="28.321" y1="0" x2="28.321" y2="22.86" width="0" layer="20"/>
 <wire x1="28.321" y1="22.86" x2="0" y2="22.86" width="0" layer="20"/>
-<text x="0.889" y="0.635" size="1.016" layer="52" font="vector" ratio="16" rot="MR90">NFC-RDBS v2.0
+<text x="0.889" y="0.635" size="1.016" layer="52" font="vector" ratio="16" rot="MR90">NFC-RDBS v2.1
 Kemere Lab
-(C)2016</text>
+(C)2017</text>
 <text x="0.635" y="15.621" size="0.762" layer="51" font="vector" ratio="16" rot="R270">STIM</text>
 <text x="27.94" y="7.874" size="1.016" layer="28" font="vector" ratio="16" rot="MR270">RTGV</text>
@@
 </class>
 </classes>
-<designrules name="Seeed_DRU *">
+<designrules name="Seeed_DRU">
 <description language="de">&lt;b&gt;EAGLE Design Rules&lt;/b&gt;
 &lt;p&gt;
@@
 <param name="rlMinPadBottom" value="10mil"/>
 <param name="rlMaxPadBottom" value="20mil"/>
-<param name="rlMinViaOuter" value="10mil"/>
+<param name="rlMinViaOuter" value="6mil"/>
 <param name="rlMaxViaOuter" value="20mil"/>
-<param name="rlMinViaInner" value="10mil"/>
+<param name="rlMinViaInner" value="6mil"/>
 <param name="rlMaxViaInner" value="20mil"/>
 <param name="rlMinMicroViaOuter" value="4mil"/>
@@
 </element>
 <element name="C2" library="rcl" package="C0603" value="0.1u" x="18.796" y="1.27" smashed="yes" rot="R180">
-<attribute name="VALUE" x="21.082" y="1.397" size="0.8128" layer="27" font="vector" ratio="16"/>
+<attribute name="VALUE" x="14.732" y="0.889" size="0.8128" layer="27" font="vector" ratio="16"/>
 </element>
 <element name="ANT" library="Samtec50Mil" package="FTSH-102-DH" value="FTSH-102" x="26.289" y="1.143" smashed="yes" rot="R180"/>
@@
 <element name="BAT1" library="Battery" package="BATTCOM_20MM_PLASTIC_STUDS" value="20mm coincell" x="16.294" y="11.557" smashed="yes" rot="MR0"/>
 <element name="C1" library="rcl" package="C0603" value="1u" x="18.796" y="2.921" smashed="yes" rot="R180">
-<attribute name="VALUE" x="21.082" y="2.667" size="0.8128" layer="27" font="vector" ratio="16"/>
+<attribute name="VALUE" x="20.828" y="2.794" size="0.8128" layer="27" font="vector" ratio="16"/>
 </element>
 <element name="C3" library="rcl" package="C1206" value="100u" x="2.794" y="5.08" smashed="yes" rot="R270">
@@
 <wire x1="24.546078125" y1="21.36255" x2="21.5791875" y2="21.36255" width="0.254" layer="1"/>
 <wire x1="21.5791875" y1="21.36255" x2="21.417034375" y2="21.200396875" width="0.254" layer="1"/>
+<contactref element="C1" pad="1"/>
+<contactref element="U$1" pad="1"/>
+<contactref element="C2" pad="1"/>
+<wire x1="21.823" y1="4.273" x2="20.998" y2="4.273" width="0.254" layer="1"/>
+<wire x1="20.998" y1="4.273" x2="19.646" y2="2.921" width="0.254" layer="1"/>
+<wire x1="20.574" y1="2.032" x2="21.678" y2="2.032" width="0.254" layer="16"/>
+<wire x1="19.685" y1="2.921" x2="19.646" y2="2.921" width="0.4064" layer="1"/>
+<wire x1="19.646" y1="2.921" x2="19.646" y2="2.032" width="0.4064" layer="1"/>
+<wire x1="19.646" y1="2.032" x2="19.646" y2="1.27" width="0.4064" layer="1"/>
+<wire x1="21.678" y1="2.032" x2="19.646" y2="2.032" width="0.4064" layer="1"/>
+<via x="21.678" y="2.032" extent="1-16" drill="0.6" shape="square"/>
+<wire x1="26.035" y1="10.414" x2="26.035" y2="6.35" width="0.254" layer="16"/>
+<wire x1="26.035" y1="6.35" x2="21.717" y2="2.032" width="0.254" layer="16"/>
+<wire x1="21.717" y1="2.032" x2="21.678" y2="2.032" width="0.254" layer="16"/>
 </signal>
 <signal name="GND">
@@
 <via x="25.908" y="15.367" extent="1-16" drill="0.6"/>
 <via x="27.051" y="4.064" extent="1-16" drill="0.6"/>
+<via x="24.003" y="1.016" extent="1-16" drill="0.6" shape="square"/>
 </signal>
 <signal name="TEST">
@@
 <wire x1="2.794" y1="11.557" x2="2.794" y2="6.48" width="0.4064" layer="1"/>
 </signal>
-<signal name="VDD2">
-<contactref element="C1" pad="1"/>
-<contactref element="U$1" pad="1"/>
-<contactref element="C2" pad="1"/>
-<wire x1="21.823" y1="4.273" x2="20.998" y2="4.273" width="0.254" layer="1"/>
-<wire x1="20.998" y1="4.273" x2="19.646" y2="2.921" width="0.254" layer="1"/>
-<wire x1="19.646" y1="2.921" x2="19.685" y2="2.921" width="0.254" layer="1"/>
-<wire x1="19.685" y1="2.921" x2="20.574" y2="2.032" width="0.254" layer="1"/>
-<wire x1="20.574" y1="2.032" x2="20.408" y2="2.032" width="0.254" layer="1"/>
-<wire x1="20.408" y1="2.032" x2="19.646" y2="1.27" width="0.254" layer="1"/>
-</signal>
 <signal name="VDD5">
