File: PCBs/Current/RatDBS-Plastic2032Battery-WithRegulator.sch (EAGLE design)
At the start: 23 parts, among them U1 LP2981-3V, U2 LP2981-5V

Commit message: Updated PCB manufacturing
Connections:
- removed net VDD2: C1.1, C2.1, U$1.VCC
- net VDD: now also C1.1, C2.1, U$1.VCC
Changed lines of the file:
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@@
 <?xml version="1.0" encoding="utf-8"?>
 <!DOCTYPE eagle SYSTEM "eagle.dtd">
-<eagle version="7.3.0">
+<eagle version="7.7.0">
 <drawing>
 <settings>
@@
 <pinref part="U1" gate="A" pin="VOUT"/>
 </segment>
+<segment>
+<pinref part="U$1" gate="G$1" pin="VCC"/>
+<wire x1="-167.64" y1="109.22" x2="-170.18" y2="109.22" width="0.1524" layer="91"/>
+<wire x1="-170.18" y1="109.22" x2="-175.26" y2="109.22" width="0.1524" layer="91"/>
+<wire x1="-175.26" y1="109.22" x2="-175.26" y2="116.84" width="0.1524" layer="91"/>
+<pinref part="VDD9" gate="G$1" pin="VDD"/>
+<pinref part="C2" gate="G$1" pin="1"/>
+<wire x1="-154.94" y1="119.38" x2="-170.18" y2="119.38" width="0.1524" layer="91"/>
+<wire x1="-170.18" y1="119.38" x2="-170.18" y2="109.22" width="0.1524" layer="91"/>
+<junction x="-170.18" y="109.22"/>
+<wire x1="-170.18" y1="119.38" x2="-170.18" y2="132.08" width="0.1524" layer="91"/>
+<wire x1="-170.18" y1="132.08" x2="-154.94" y2="132.08" width="0.1524" layer="91"/>
+<junction x="-170.18" y="119.38"/>
+<pinref part="C1" gate="G$1" pin="1"/>
+</segment>
 </net>
 <net name="GND" class="0">
@@
 <junction x="-213.36" y="48.26"/>
 <pinref part="C3" gate="G$1" pin="1"/>
+<junction x="-200.66" y="48.26"/>
 </segment>
 <segment>
@@
 </segment>
 </net>
-<net name="VDD2" class="0">
-<segment>
-<pinref part="U$1" gate="G$1" pin="VCC"/>
-<wire x1="-167.64" y1="109.22" x2="-170.18" y2="109.22" width="0.1524" layer="91"/>
-<wire x1="-170.18" y1="109.22" x2="-175.26" y2="109.22" width="0.1524" layer="91"/>
-<wire x1="-175.26" y1="109.22" x2="-175.26" y2="116.84" width="0.1524" layer="91"/>
-<pinref part="VDD9" gate="G$1" pin="VDD"/>
-<pinref part="C2" gate="G$1" pin="1"/>
-<wire x1="-154.94" y1="119.38" x2="-170.18" y2="119.38" width="0.1524" layer="91"/>
-<wire x1="-170.18" y1="119.38" x2="-170.18" y2="109.22" width="0.1524" layer="91"/>
-<junction x="-170.18" y="109.22"/>
-<wire x1="-170.18" y1="119.38" x2="-170.18" y2="132.08" width="0.1524" layer="91"/>
-<wire x1="-170.18" y1="132.08" x2="-154.94" y2="132.08" width="0.1524" layer="91"/>
-<junction x="-170.18" y="119.38"/>
-<pinref part="C1" gate="G$1" pin="1"/>
-</segment>
-</net>
