File: PCBs/Current/RatDBS-TrackBattery.brd (EAGLE design)
At the start: 28.3 x 22.9 mm, 27 parts, among them U1 3V, U2 5V

Commit message: Added resistor values for voltage divider and LEDs. Labeled preferred 332 inductor antenna and CANT values.
Parts:
- ANT: value FTSH-102 -> 3.3uH
- CANT: value C_NFC -> 8pF
- RDIV_HIGH: value RDIV_HIGH -> 20k
- RDIV_LOW: value RDIV_LOW -> 10k
- R_LEDG: value R_LEDG -> 10k
- R_LEDR: value R_LEDR -> 10k
- renumbered RDIV_1 to RDIV_HIGH, RDIV_2 to RDIV_LOW, R_LED to R_LEDR, R_LED1 to R_LEDG
Changed lines of the file:
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@@
 <?xml version="1.0" encoding="utf-8"?>
 <!DOCTYPE eagle SYSTEM "eagle.dtd">
-<eagle version="7.7.0">
+<eagle version="8.2.2">
 <drawing>
 <settings>
@@
 <attribute name="VALUE" x="24.892" y="21.971" size="0.8128" layer="27" font="vector" ratio="16" rot="R180"/>
 </element>
-<element name="R_LED" library="BiphasicBoard" package="R0603" value="R_LEDR" x="15.748" y="3.556" smashed="yes" rot="MR270">
+<element name="R_LEDR" library="BiphasicBoard" package="R0603" value="10k" x="15.748" y="3.556" smashed="yes" rot="MR270">
 <attribute name="VALUE" x="17.653" y="5.842" size="0.8128" layer="28" font="vector" ratio="16" rot="MR270"/>
 </element>
@@
 <attribute name="VALUE" x="8.382" y="13.97" size="0.8128" layer="27" font="vector" ratio="16"/>
 </element>
-<element name="ANT" library="Samtec50Mil" package="FTSH-102-DH" value="FTSH-102" x="1.397" y="18.923" smashed="yes" rot="R90"/>
-<element name="CANT" library="rcl" package="C0603" value="C_NFC" x="2.667" y="18.923" smashed="yes" rot="MR90">
+<element name="ANT" library="Samtec50Mil" package="FTSH-102-DH" value="3.3uH" x="1.397" y="18.923" smashed="yes" rot="R90"/>
+<element name="CANT" library="rcl" package="C0603" value="8pF" x="2.667" y="18.923" smashed="yes" rot="MR90">
 <attribute name="VALUE" x="3.683" y="16.891" size="0.8128" layer="28" font="vector" ratio="16" rot="MR90"/>
 </element>
@@
 </element>
 <element name="U1" library="Texas Instruments_By_element14_Batch_1" package="SOT95P280X145-5N" value="3V" x="4.064" y="5.461" smashed="yes" rot="MR180">
+<attribute name="MPN" value="LP2985A-33DBVTE4" x="4.064" y="5.461" size="1.778" layer="28" rot="MR180" display="off"/>
+<attribute name="OC_FARNELL" value="1053660" x="4.064" y="5.461" size="1.778" layer="28" rot="MR180" display="off"/>
+<attribute name="OC_NEWARK" value="79K3928" x="4.064" y="5.461" size="1.778" layer="28" rot="MR180" display="off"/>
 <attribute name="PACKAGE" value="SOT-23-5" x="4.064" y="5.461" size="1.778" layer="28" rot="MR180" display="off"/>
-<attribute name="OC_FARNELL" value="1053660" x="4.064" y="5.461" size="1.778" layer="28" rot="MR180" display="off"/>
 <attribute name="SUPPLIER" value="Texas Instruments" x="4.064" y="5.461" size="1.778" layer="28" rot="MR180" display="off"/>
-<attribute name="MPN" value="LP2985A-33DBVTE4" x="4.064" y="5.461" size="1.778" layer="28" rot="MR180" display="off"/>
-<attribute name="OC_NEWARK" value="79K3928" x="4.064" y="5.461" size="1.778" layer="28" rot="MR180" display="off"/>
 <attribute name="VALUE" x="3.4036" y="3.556" size="0.8128" layer="28" font="vector" ratio="16" rot="SMR180"/>
 </element>
 <element name="U2" library="Texas Instruments_By_element14_Batch_1" package="SOT95P280X145-5N" value="5V" x="5.969" y="13.208" smashed="yes" rot="MR90">
+<attribute name="MPN" value="LP2985A-33DBVTE4" x="5.969" y="13.208" size="1.778" layer="28" rot="MR90" display="off"/>
 <attribute name="OC_FARNELL" value="1053660" x="5.969" y="13.208" size="1.778" layer="28" rot="MR90" display="off"/>
-<attribute name="MPN" value="LP2985A-33DBVTE4" x="5.969" y="13.208" size="1.778" layer="28" rot="MR90" display="off"/>
+<attribute name="OC_NEWARK" value="79K3928" x="5.969" y="13.208" size="1.778" layer="28" rot="MR90" display="off"/>
 <attribute name="PACKAGE" value="SOT-23-5" x="5.969" y="13.208" size="1.778" layer="28" rot="MR90" display="off"/>
-<attribute name="OC_NEWARK" value="79K3928" x="5.969" y="13.208" size="1.778" layer="28" rot="MR90" display="off"/>
 <attribute name="SUPPLIER" value="Texas Instruments" x="5.969" y="13.208" size="1.778" layer="28" rot="MR90" display="off"/>
 <attribute name="VALUE" x="8.763" y="13.8684" size="0.8128" layer="28" font="vector" ratio="16" rot="SMR270"/>
@@
 <attribute name="VALUE" x="22.022503125" y="8.970775" size="0.8128" layer="27" font="vector" ratio="16" rot="R270"/>
 </element>
-<element name="RDIV_2" library="BiphasicBoard" package="R0603" value="RDIV_LOW" x="8.89" y="8.763" smashed="yes" rot="MR180">
+<element name="RDIV_LOW" library="BiphasicBoard" package="R0603" value="10k" x="8.89" y="8.763" smashed="yes" rot="MR180">
 <attribute name="VALUE" x="10.414" y="9.144" size="0.8128" layer="28" font="vector" ratio="16" rot="MR180"/>
 </element>
-<element name="RDIV_1" library="BiphasicBoard" package="R0603" value="RDIV_HIGH" x="8.89" y="10.16" smashed="yes" rot="MR180">
+<element name="RDIV_HIGH" library="BiphasicBoard" package="R0603" value="20k" x="8.89" y="10.16" smashed="yes" rot="MR180">
 <attribute name="VALUE" x="10.414" y="10.541" size="0.8128" layer="28" font="vector" ratio="16" rot="MR180"/>
 </element>
-<element name="R_LED1" library="BiphasicBoard" package="R0603" value="R_LEDG" x="13.5255" y="3.556" smashed="yes" rot="MR270">
+<element name="R_LEDG" library="BiphasicBoard" package="R0603" value="10k" x="13.5255" y="3.556" smashed="yes" rot="MR270">
 <attribute name="VALUE" x="12.5095" y="5.842" size="0.8128" layer="28" font="vector" ratio="16" rot="MR270"/>
 </element>
@@
 </polygon>
 <contactref element="C4" pad="2"/>
-<contactref element="RDIV_2" pad="1"/>
+<contactref element="RDIV_LOW" pad="1"/>
 <contactref element="LED1" pad="C"/>
 <via x="12.065" y="4.699" extent="1-16" drill="0.3048" shape="square"/>
@@
 <signal name="N$5">
 <contactref element="MSP430" pad="13"/>
-<contactref element="R_LED" pad="1"/>
+<contactref element="R_LEDR" pad="1"/>
 <wire x1="15.748" y1="4.406" x2="15.494" y2="4.191" width="0.254" layer="16"/>
 <wire x1="15.494" y1="4.191" x2="14.605" y2="4.191" width="0.254" layer="16"/>
@@
 </signal>
 <signal name="N$9">
-<contactref element="R_LED" pad="2"/>
+<contactref element="R_LEDR" pad="2"/>
 <contactref element="LED6" pad="A"/>
 <wire x1="15.748" y1="2.706" x2="15.748" y2="1.651" width="0.254" layer="16"/>
@@
 <contactref element="U2" pad="3"/>
 <contactref element="C3" pad="1"/>
-<contactref element="RDIV_1" pad="1"/>
+<contactref element="RDIV_HIGH" pad="1"/>
 <wire x1="8.04" y1="10.16" x2="6.9088" y2="10.795" width="0.4064" layer="16"/>
 <wire x1="6.9088" y1="10.795" x2="5.0292" y2="10.795" width="0.4064" layer="16"/>
@@
 <signal name="N$10">
 <contactref element="MSP430" pad="6"/>
-<contactref element="RDIV_2" pad="2"/>
-<contactref element="RDIV_1" pad="2"/>
+<contactref element="RDIV_LOW" pad="2"/>
+<contactref element="RDIV_HIGH" pad="2"/>
 <wire x1="15.4865" y1="10.3296" x2="15.494" y2="10.3296" width="0.254" layer="1"/>
 <wire x1="15.494" y1="10.3296" x2="15.494" y2="9.017" width="0.254" layer="1"/>
@@
 <signal name="N$11">
 <contactref element="MSP430" pad="12"/>
-<contactref element="R_LED1" pad="1"/>
+<contactref element="R_LEDG" pad="1"/>
 <via x="13.5255" y="5.588" extent="1-16" drill="0.3048" shape="square"/>
 <wire x1="13.5255" y1="4.406" x2="13.5255" y2="5.588" width="0.254" layer="16"/>
@@
 </signal>
 <signal name="N$13">
-<contactref element="R_LED1" pad="2"/>
+<contactref element="R_LEDG" pad="2"/>
 <contactref element="LED1" pad="A"/>
 <wire x1="5.056" y1="1.651" x2="5.056" y2="1.69" width="0.254" layer="1"/>
